File: PCB/Curse_PCB/Curse_PCB.sch (KiCad schematic (older format))
At the start: 14 parts

Commit message: SCH + PCB
Parts:
- removed TP1: 32.768 kHz TP, TestPoint:TestPoint_THTPad_D1.0mm_Drill0.5mm, symbol Connector:TestPoint
- added XP4: I2C_SENSOR_CONN, Connector_PinHeader_2.54mm:PinHeader_1x04_P2.54mm_Vertical, symbol Connector_Generic:Conn_01x04
- added XP7: ADC1_CONN, Connector_PinHeader_2.54mm:PinHeader_1x03_P2.54mm_Vertical, symbol Connector_Generic:Conn_01x03
- BQ1: footprint Crystal:Crystal_DS26_D2.0mm_L6.0mm_Horizontal -> Crystal:Crystal_SMD_3215-2Pin_3.2x1.5mm
- R1, R2: value 47K -> 10K
Connections:
- net labels added: ADC_CH6, ADC_CH7, SCL, SDA
- wire segments 29 -> 28

Commit message: АЦП
Parts:
- removed XP7: ADC1_CONN, Connector_PinHeader_2.54mm:PinHeader_1x03_P2.54mm_Vertical, symbol Connector_Generic:Conn_01x03
- added R5, R6: 10K, Resistor_SMD:R_0603_1608Metric, symbol Device:R
- XP1: footprint Connector_PinHeader_2.54mm:PinHeader_1x02_P2.54mm_Vertical -> Connector_PinHeader_2.54mm:PinHeader_1x03_P2.54mm_Vertical; symbol Connector_Generic:Conn_01x02 -> Connector_Generic:Conn_01x03
Connections:
- net labels added: BAT_ADC, DS18B20
- net labels removed: ADC_CH6, ADC_CH7
- wire segments 28 -> 31
Other:
- note added: "V_BAT/2"
Changed lines of the file:
@@
 L Connector_Generic:Conn_01x08 XP3
 U 1 1 6163EBFE
-P 4300 7200
-F 0 "XP3" H 4218 6575 50  0000 C CNN
-F 1 "ESP_CONN" H 4218 6666 50  0000 C CNN
-F 2 "Connector_PinSocket_2.54mm:PinSocket_2x04_P2.54mm_Vertical" H 4300 7200 50  0001 C CNN
-F 3 "~" H 4300 7200 50  0001 C CNN
-	1    4300 7200
+P 4350 6600
+F 0 "XP3" H 4268 5975 50  0000 C CNN
+F 1 "ESP_CONN" H 4268 6066 50  0000 C CNN
+F 2 "Connector_PinSocket_2.54mm:PinSocket_2x04_P2.54mm_Vertical" H 4350 6600 50  0001 C CNN
+F 3 "~" H 4350 6600 50  0001 C CNN
+	1    4350 6600
 	-1   0    0    1
 $EndComp
@@
 L power:+3V3 #PWR0107
 U 1 1 616420BD
-P 4500 7100
-F 0 "#PWR0107" H 4500 6950 50  0001 C CNN
-F 1 "+3V3" V 4515 7228 50  0000 L CNN
-F 2 "" H 4500 7100 50  0001 C CNN
-F 3 "" H 4500 7100 50  0001 C CNN
-	1    4500 7100
+P 4550 6500
+F 0 "#PWR0107" H 4550 6350 50  0001 C CNN
+F 1 "+3V3" V 4565 6628 50  0000 L CNN
+F 2 "" H 4550 6500 50  0001 C CNN
+F 3 "" H 4550 6500 50  0001 C CNN
+	1    4550 6500
 	0    1    1    0
 $EndComp
@@
 L power:GND #PWR0108
 U 1 1 616435D8
-P 4500 7500
-F 0 "#PWR0108" H 4500 7250 50  0001 C CNN
-F 1 "GND" H 4505 7327 50  0000 C CNN
-F 2 "" H 4500 7500 50  0001 C CNN
-F 3 "" H 4500 7500 50  0001 C CNN
-	1    4500 7500
+P 4550 6900
+F 0 "#PWR0108" H 4550 6650 50  0001 C CNN
+F 1 "GND" H 4555 6727 50  0000 C CNN
+F 2 "" H 4550 6900 50  0001 C CNN
+F 3 "" H 4550 6900 50  0001 C CNN
+	1    4550 6900
 	0    -1   -1   0
 $EndComp
@@
 $EndComp
 $Comp
-L Connector_Generic:Conn_01x02 XP1
-U 1 1 616597E9
-P 4425 3300
-F 0 "XP1" H 4505 3292 50  0000 L CNN
-F 1 "POWER_CONN" H 4505 3201 50  0000 L CNN
-F 2 "Connector_PinHeader_2.54mm:PinHeader_1x02_P2.54mm_Vertical" H 4425 3300 50  0001 C CNN
-F 3 "~" H 4425 3300 50  0001 C CNN
-	1    4425 3300
-	1    0    0    -1
-$EndComp
-$Comp
 L power:+3V3 #PWR0115
 U 1 1 6165A797
-P 4225 3300
-F 0 "#PWR0115" H 4225 3150 50  0001 C CNN
-F 1 "+3V3" V 4240 3428 50  0000 L CNN
-F 2 "" H 4225 3300 50  0001 C CNN
-F 3 "" H 4225 3300 50  0001 C CNN
-	1    4225 3300
-	0    -1   -1   0
-$EndComp
-$Comp
-L power:GND #PWR0116
-U 1 1 6165BD45
-P 4225 3400
-F 0 "#PWR0116" H 4225 3150 50  0001 C CNN
-F 1 "GND" H 4230 3227 50  0000 C CNN
-F 2 "" H 4225 3400 50  0001 C CNN
-F 3 "" H 4225 3400 50  0001 C CNN
-	1    4225 3400
-	1    0    0    -1
+P 3725 3450
+F 0 "#PWR0115" H 3725 3300 50  0001 C CNN
+F 1 "+3V3" V 3740 3578 50  0000 L CNN
+F 2 "" H 3725 3450 50  0001 C CNN
+F 3 "" H 3725 3450 50  0001 C CNN
+	1    3725 3450
+	0    1    1    0
 $EndComp
 Text Label 5975 4625 0    50   ~ 0
@@
 Text Label 5975 4725 0    50   ~ 0
 UART_RX
-Text Label 4500 7200 0    50   ~ 0
+Text Label 4550 6600 0    50   ~ 0
 UART_TX
-Text Label 4500 6800 0    50   ~ 0
+Text Label 4550 6200 0    50   ~ 0
 UART_RX
 Wire Wire Line
@@
 Text Label 4550 5000 0    50   ~ 0
 SDA
-Text Label 6500 4825 2    50   ~ 0
-ADC_CH6
+Text Label 8900 5475 0    50   ~ 0
+DS18B20
 Text Label 4550 5725 0    50   ~ 0
-ADC_CH6
-$Comp
-L Connector_Generic:Conn_01x03 XP7
-U 1 1 61689B2D
-P 4350 6225
-F 0 "XP7" H 4430 6267 50  0000 L CNN
-F 1 "ADC1_CONN" H 4430 6176 50  0000 L CNN
-F 2 "Connector_PinHeader_2.54mm:PinHeader_1x03_P2.54mm_Vertical" H 4350 6225 50  0001 C CNN
-F 3 "~" H 4350 6225 50  0001 C CNN
-	1    4350 6225
-	-1   0    0    1
-$EndComp
-$Comp
-L power:+3V3 #PWR0120
-U 1 1 61689B33
-P 4550 6325
-F 0 "#PWR0120" H 4550 6175 50  0001 C CNN
-F 1 "+3V3" V 4565 6453 50  0000 L CNN
-F 2 "" H 4550 6325 50  0001 C CNN
-F 3 "" H 4550 6325 50  0001 C CNN
-	1    4550 6325
-	0    1    1    0
-$EndComp
-$Comp
-L power:GND #PWR0121
-U 1 1 61689B39
-P 4550 6125
-F 0 "#PWR0121" H 4550 5875 50  0001 C CNN
-F 1 "GND" H 4555 5952 50  0000 C CNN
-F 2 "" H 4550 6125 50  0001 C CNN
-F 3 "" H 4550 6125 50  0001 C CNN
-	1    4550 6125
-	-1   0    0    1
-$EndComp
-Text Label 4550 6225 0    50   ~ 0
-ADC_CH7
-Text Label 6500 4925 2    50   ~ 0
-ADC_CH7
+DS18B20
+Text Label 8900 5375 0    50   ~ 0
+BAT_ADC
+$Comp
+L Device:R R5
+U 1 1 6165AADB
+P 4300 3425
+F 0 "R5" H 4370 3471 50  0000 L CNN
+F 1 "10K" H 4370 3380 50  0000 L CNN
+F 2 "Resistor_SMD:R_0603_1608Metric" V 4230 3425 50  0001 C CNN
+F 3 "~" H 4300 3425 50  0001 C CNN
+	1    4300 3425
+	1    0    0    -1
+$EndComp
+$Comp
+L Device:R R6
+U 1 1 6165B739
+P 4750 3250
+F 0 "R6" H 4820 3296 50  0000 L CNN
+F 1 "10K" H 4820 3205 50  0000 L CNN
+F 2 "Resistor_SMD:R_0603_1608Metric" V 4680 3250 50  0001 C CNN
+F 3 "~" H 4750 3250 50  0001 C CNN
+	1    4750 3250
+	0    -1   -1   0
+$EndComp
+$Comp
+L power:GND #PWR01
+U 1 1 6165CBC1
+P 4300 3575
+F 0 "#PWR01" H 4300 3325 50  0001 C CNN
+F 1 "GND" H 4305 3402 50  0000 C CNN
+F 2 "" H 4300 3575 50  0001 C CNN
+F 3 "" H 4300 3575 50  0001 C CNN
+	1    4300 3575
+	1    0    0    -1
+$EndComp
+Wire Wire Line
+	3725 3250 4300 3250
+Wire Wire Line
+	4300 3275 4300 3250
+Connection ~ 4300 3250
+Wire Wire Line
+	4300 3250 4600 3250
+Text Label 4900 3250 0    50   ~ 0
+BAT_ADC
+Wire Notes Line
+	4600 3050 3950 3050
+Text Notes 3950 3200 0    100  Italic 0
+V_BAT/2
+Wire Notes Line
+	4600 3050 4600 3225
+Wire Notes Line
+	4600 3225 3950 3225
+Wire Notes Line
+	3950 3225 3950 3050
+$Comp
+L power:GND #PWR0116
+U 1 1 6165BD45
+P 3725 3350
+F 0 "#PWR0116" H 3725 3100 50  0001 C CNN
+F 1 "GND" H 3730 3177 50  0000 C CNN
+F 2 "" H 3725 3350 50  0001 C CNN
+F 3 "" H 3725 3350 50  0001 C CNN
+	1    3725 3350
+	0    -1   -1   0
+$EndComp
+$Comp
+L Connector_Generic:Conn_01x03 XP1
+U 1 1 616597E9
+P 3525 3350
+F 0 "XP1" H 3605 3342 50  0000 L CNN
+F 1 "POWER_CONN" H 3605 3251 50  0000 L CNN
+F 2 "Connector_PinHeader_2.54mm:PinHeader_1x03_P2.54mm_Vertical" H 3525 3350 50  0001 C CNN
+F 3 "~" H 3525 3350 50  0001 C CNN
+	1    3525 3350
+	-1   0    0    1
+$EndComp
 $EndSCHEMATC

Commit message: LDO
Parts:
- added C3, C4: 10 uF, Capacitor_SMD:C_0603_1608Metric, symbol Device:C
- added DA1: AMS1117-3.3, Package_TO_SOT_SMD:SOT-223-3_TabPin2, symbol Regulator_Linear:AMS1117-3.3
Connections:
- net labels added: +5V
- wire segments 31 -> 39
Changed lines of the file:
@@
 L power:+3V3 #PWR0115
 U 1 1 6165A797
-P 3725 3450
-F 0 "#PWR0115" H 3725 3300 50  0001 C CNN
-F 1 "+3V3" V 3740 3578 50  0000 L CNN
-F 2 "" H 3725 3450 50  0001 C CNN
-F 3 "" H 3725 3450 50  0001 C CNN
-	1    3725 3450
+P 4775 3075
+F 0 "#PWR0115" H 4775 2925 50  0001 C CNN
+F 1 "+3V3" V 4790 3203 50  0000 L CNN
+F 2 "" H 4775 3075 50  0001 C CNN
+F 3 "" H 4775 3075 50  0001 C CNN
+	1    4775 3075
 	0    1    1    0
 $EndComp
@@
 Text Label 4550 5725 0    50   ~ 0
 DS18B20
-Text Label 8900 5375 0    50   ~ 0
+Text Label 8900 4975 0    50   ~ 0
 BAT_ADC
 $Comp
 L Device:R R5
 U 1 1 6165AADB
-P 4300 3425
-F 0 "R5" H 4370 3471 50  0000 L CNN
-F 1 "10K" H 4370 3380 50  0000 L CNN
-F 2 "Resistor_SMD:R_0603_1608Metric" V 4230 3425 50  0001 C CNN
-F 3 "~" H 4300 3425 50  0001 C CNN
-	1    4300 3425
+P 3800 2150
+F 0 "R5" H 3870 2196 50  0000 L CNN
+F 1 "10K" H 3870 2105 50  0000 L CNN
+F 2 "Resistor_SMD:R_0603_1608Metric" V 3730 2150 50  0001 C CNN
+F 3 "~" H 3800 2150 50  0001 C CNN
+	1    3800 2150
 	1    0    0    -1
 $EndComp
@@
 L Device:R R6
 U 1 1 6165B739
-P 4750 3250
-F 0 "R6" H 4820 3296 50  0000 L CNN
-F 1 "10K" H 4820 3205 50  0000 L CNN
-F 2 "Resistor_SMD:R_0603_1608Metric" V 4680 3250 50  0001 C CNN
-F 3 "~" H 4750 3250 50  0001 C CNN
-	1    4750 3250
+P 4250 1975
+F 0 "R6" H 4320 2021 50  0000 L CNN
+F 1 "10K" H 4320 1930 50  0000 L CNN
+F 2 "Resistor_SMD:R_0603_1608Metric" V 4180 1975 50  0001 C CNN
+F 3 "~" H 4250 1975 50  0001 C CNN
+	1    4250 1975
 	0    -1   -1   0
 $EndComp
@@
 L power:GND #PWR01
 U 1 1 6165CBC1
-P 4300 3575
-F 0 "#PWR01" H 4300 3325 50  0001 C CNN
-F 1 "GND" H 4305 3402 50  0000 C CNN
-F 2 "" H 4300 3575 50  0001 C CNN
-F 3 "" H 4300 3575 50  0001 C CNN
-	1    4300 3575
-	1    0    0    -1
-$EndComp
-Wire Wire Line
-	3725 3250 4300 3250
-Wire Wire Line
-	4300 3275 4300 3250
-Connection ~ 4300 3250
-Wire Wire Line
-	4300 3250 4600 3250
-Text Label 4900 3250 0    50   ~ 0
+P 3800 2300
+F 0 "#PWR01" H 3800 2050 50  0001 C CNN
+F 1 "GND" H 3805 2127 50  0000 C CNN
+F 2 "" H 3800 2300 50  0001 C CNN
+F 3 "" H 3800 2300 50  0001 C CNN
+	1    3800 2300
+	1    0    0    -1
+$EndComp
+Wire Wire Line
+	3225 1975 3800 1975
+Wire Wire Line
+	3800 2000 3800 1975
+Connection ~ 3800 1975
+Wire Wire Line
+	3800 1975 4100 1975
+Text Label 4400 1975 0    50   ~ 0
 BAT_ADC
 Wire Notes Line
-	4600 3050 3950 3050
-Text Notes 3950 3200 0    100  Italic 0
+	4100 1775 3450 1775
+Text Notes 3450 1925 0    100  Italic 0
 V_BAT/2
 Wire Notes Line
-	4600 3050 4600 3225
+	4100 1775 4100 1950
 Wire Notes Line
-	4600 3225 3950 3225
+	4100 1950 3450 1950
 Wire Notes Line
-	3950 3225 3950 3050
+	3450 1950 3450 1775
 $Comp
 L power:GND #PWR0116
 U 1 1 6165BD45
-P 3725 3350
-F 0 "#PWR0116" H 3725 3100 50  0001 C CNN
-F 1 "GND" H 3730 3177 50  0000 C CNN
-F 2 "" H 3725 3350 50  0001 C CNN
-F 3 "" H 3725 3350 50  0001 C CNN
-	1    3725 3350
+P 3225 2075
+F 0 "#PWR0116" H 3225 1825 50  0001 C CNN
+F 1 "GND" H 3230 1902 50  0000 C CNN
+F 2 "" H 3225 2075 50  0001 C CNN
+F 3 "" H 3225 2075 50  0001 C CNN
+	1    3225 2075
 	0    -1   -1   0
 $EndComp
@@
 L Connector_Generic:Conn_01x03 XP1
 U 1 1 616597E9
-P 3525 3350
-F 0 "XP1" H 3605 3342 50  0000 L CNN
-F 1 "POWER_CONN" H 3605 3251 50  0000 L CNN
-F 2 "Connector_PinHeader_2.54mm:PinHeader_1x03_P2.54mm_Vertical" H 3525 3350 50  0001 C CNN
-F 3 "~" H 3525 3350 50  0001 C CNN
-	1    3525 3350
+P 3025 2075
+F 0 "XP1" H 3105 2067 50  0000 L CNN
+F 1 "POWER_CONN" H 3105 1976 50  0000 L CNN
+F 2 "Connector_PinHeader_2.54mm:PinHeader_1x03_P2.54mm_Vertical" H 3025 2075 50  0001 C CNN
+F 3 "~" H 3025 2075 50  0001 C CNN
+	1    3025 2075
 	-1   0    0    1
 $EndComp
+$Comp
+L Regulator_Linear:AMS1117-3.3 DA1
+U 1 1 6165B979
+P 3900 3075
+F 0 "DA1" H 3900 3317 50  0000 C CNN
+F 1 "AMS1117-3.3" H 3900 3226 50  0000 C CNN
+F 2 "Package_TO_SOT_SMD:SOT-223-3_TabPin2" H 3900 3275 50  0001 C CNN
+F 3 "http://www.advanced-monolithic.com/pdf/ds1117.pdf" H 4000 2825 50  0001 C CNN
+	1    3900 3075
+	1    0    0    -1
+$EndComp
+Wire Wire Line
+	4200 3075 4425 3075
+$Comp
+L power:+5V #PWR03
+U 1 1 6165F30A
+P 3225 2175
+F 0 "#PWR03" H 3225 2025 50  0001 C CNN
+F 1 "+5V" H 3240 2348 50  0000 C CNN
+F 2 "" H 3225 2175 50  0001 C CNN
+F 3 "" H 3225 2175 50  0001 C CNN
+	1    3225 2175
+	0    1    1    0
+$EndComp
+$Comp
+L power:+5V #PWR02
+U 1 1 61662FAF
+P 3075 2950
+F 0 "#PWR02" H 3075 2800 50  0001 C CNN
+F 1 "+5V" H 3090 3123 50  0000 C CNN
+F 2 "" H 3075 2950 50  0001 C CNN
+F 3 "" H 3075 2950 50  0001 C CNN
+	1    3075 2950
+	1    0    0    -1
+$EndComp
+Wire Wire Line
+	3075 2950 3075 3075
+Wire Wire Line
+	3075 3075 3350 3075
+$Comp
+L Device:C C3
+U 1 1 616645A1
+P 3350 3300
+F 0 "C3" H 3465 3346 50  0000 L CNN
+F 1 "10 uF" H 3465 3255 50  0000 L CNN
+F 2 "Capacitor_SMD:C_0603_1608Metric" H 3388 3150 50  0001 C CNN
+F 3 "~" H 3350 3300 50  0001 C CNN
+	1    3350 3300
+	1    0    0    -1
+$EndComp
+$Comp
+L Device:C C4
+U 1 1 616650FC
+P 4425 3300
+F 0 "C4" H 4540 3346 50  0000 L CNN
+F 1 "10 uF" H 4540 3255 50  0000 L CNN
+F 2 "Capacitor_SMD:C_0603_1608Metric" H 4463 3150 50  0001 C CNN
+F 3 "~" H 4425 3300 50  0001 C CNN
+	1    4425 3300
+	1    0    0    -1
+$EndComp
+$Comp
+L power:GND #PWR05
+U 1 1 61665BEB
+P 3900 3450
+F 0 "#PWR05" H 3900 3200 50  0001 C CNN
+F 1 "GND" H 3905 3277 50  0000 C CNN
+F 2 "" H 3900 3450 50  0001 C CNN
+F 3 "" H 3900 3450 50  0001 C CNN
+	1    3900 3450
+	1    0    0    -1
+$EndComp
+$Comp
+L power:GND #PWR04
+U 1 1 61666433
+P 3350 3450
+F 0 "#PWR04" H 3350 3200 50  0001 C CNN
+F 1 "GND" H 3355 3277 50  0000 C CNN
+F 2 "" H 3350 3450 50  0001 C CNN
+F 3 "" H 3350 3450 50  0001 C CNN
+	1    3350 3450
+	1    0    0    -1
+$EndComp
+$Comp
+L power:GND #PWR06
+U 1 1 61666C76
+P 4425 3450
+F 0 "#PWR06" H 4425 3200 50  0001 C CNN
+F 1 "GND" H 4430 3277 50  0000 C CNN
+F 2 "" H 4425 3450 50  0001 C CNN
+F 3 "" H 4425 3450 50  0001 C CNN
+	1    4425 3450
+	1    0    0    -1
+$EndComp
+Wire Wire Line
+	4425 3150 4425 3075
+Connection ~ 4425 3075
+Wire Wire Line
+	4425 3075 4775 3075
+Wire Wire Line
+	3350 3150 3350 3075
+Connection ~ 3350 3075
+Wire Wire Line
+	3350 3075 3600 3075
+Wire Wire Line
+	3900 3375 3900 3450
 $EndSCHEMATC

Commit message: схема
Parts:
- removed BQ1: Crystal, Crystal:Crystal_SMD_3215-2Pin_3.2x1.5mm, symbol Device:Crystal
- removed C1: 0.1 uF, Capacitor_SMD:C_0603_1608Metric, symbol Device:C
- removed C2: 2200 pF, Capacitor_SMD:C_0603_1608Metric, symbol Device:C
- removed C3, C4: 10 uF, Capacitor_SMD:C_0603_1608Metric, symbol Device:C
- removed DA1: AMS1117-3.3, Package_TO_SOT_SMD:SOT-223-3_TabPin2, symbol Regulator_Linear:AMS1117-3.3
- removed DD1: MSP430F2112IPW, Package_SO:TSSOP-28_4.4x9.7mm_P0.65mm, symbol MCU_Texas_MSP430:MSP430F2112IPW
- removed R1, R2, R5, R6: 10K, Resistor_SMD:R_0603_1608Metric, symbol Device:R
- removed R3, R4: 47K, Resistor_SMD:R_0603_1608Metric, symbol Device:R
- removed XP1: POWER_CONN, Connector_PinHeader_2.54mm:PinHeader_1x03_P2.54mm_Vertical, symbol Connector_Generic:Conn_01x03
- removed XP2: DISP_CONN, Connector_PinHeader_2.54mm:PinHeader_1x04_P2.54mm_Vertical, symbol Connector_Generic:Conn_01x04
- removed XP3: ESP_CONN, Connector_PinSocket_2.54mm:PinSocket_2x04_P2.54mm_Vertical, symbol Connector_Generic:Conn_01x08
- removed XP4: I2C_SENSOR_CONN, Connector_PinHeader_2.54mm:PinHeader_1x04_P2.54mm_Vertical, symbol Connector_Generic:Conn_01x04
- removed XP5: ADC0_CONN, Connector_PinHeader_2.54mm:PinHeader_1x03_P2.54mm_Vertical, symbol Connector_Generic:Conn_01x03
- removed XP6: BTN_CONN, Connector_PinHeader_2.54mm:PinHeader_1x02_P2.54mm_Vertical, symbol Connector_Generic:Conn_01x02
- added C? (x2): 0.1 мкФ, Capacitor_SMD:C_0603_1608Metric, symbol Device_GOST:C
- added C?: 2200 пФ, Capacitor_SMD:C_0603_1608Metric, symbol Device_GOST:C
- added C? (x3): 10 мкФ, Capacitor_SMD:C_0805_2012Metric, symbol Device_GOST:C
- added DA?: TPS63031, Package_SON:WSON-10-1EP_2.5x2.5mm_P0.5mm_EP1.2x2mm_ThermalVias, symbol My_Lib_GOST:TPS6303x
- added DD?: MSP430F2112, Package_SO:TSSOP-28_4.4x9.7mm_P0.65mm, symbol My_Lib_GOST:MSP430F21x2
- added GB?: GB_BATTERY, Battery:BatteryHolder_Keystone_1042_1x18650, symbol KGL_Power:GB_BATTERY
- added L?: 1,5 мкГн, symbol Device_GOST:L_INDUCTOR
- added R?: 47 кОм, Resistor_SMD:R_0603_1608Metric, symbol Device_GOST:R
- added R? (x4): 10 кОм, Resistor_SMD:R_0603_1608Metric, symbol Device_GOST:R
- added R?: 100 кОм, symbol Device_GOST:R
- added SA?: SA_SPST_NO, Button_Switch_THT:SW_Tactile_SPST_Angled_PTS645Vx58-2LFS, symbol Device_GOST:SA_SPST_NO
- added XS? (x2): CONN_4, symbol Connector_Generic_GOST:CONN_4
- added XS?: CONN_8, symbol Connector_Generic_GOST:CONN_8
- added ZQ?: 32 kHz, symbol Device_GOST:ZQ_CRYSTAL
Connections:
- net labels added: +3.3V
- net labels removed: +3V3, +5V, BTN0, DS18B20
- wire segments 39 -> 87
Other:
- note removed: "V_BAT/2"

Commit message: sch
Parts:
- added C1: 0.1 мкФ, Capacitor_SMD:C_0603_1608Metric, symbol Device_GOST:C
- added DA1: BQ29737, Package_SON:WSON-6_1.5x1.5mm_P0.5mm, symbol My_Lib_GOST:BQ297xx
- added R1: 330 Ом, Resistor_SMD:R_0603_1608Metric, symbol Device_GOST:R
- added R2: 2,2 кОм, Resistor_SMD:R_0603_1608Metric, symbol Device_GOST:R
- added VT1: BUK9K5R1-30E, Package_TO_SOT_SMD:LFPAK56D, symbol My_Lib_GOST:BUK9K5R1-30E
- gave numbers to parts that had none: 21
Connections:
- net EXP: now also R2.2, VT1.1 (S1); no longer GB01.2 (-)
- net at DD1.24 (P1.3): now also R5.1, SA1.1
- net ESP_IO2: now reaches DD1.26 (P1.5)
- net ESP_IO2: now also XS1.2
- net ESP_CH_PD: now reaches DD1.27 (P1.6)
- net ESP_CH_PD: now also XS1.6
- net ESP_REST: now reaches DD1.28 (P1.7)
- net ESP_REST: now also XS1.7
- net at C2.1, DA2.5 (VIN): now also GB01.1 (+), R3.1, R4.1, R1.1
- net ESP_IO0: now reaches XS1.3
- net ESP_IO0: now also DD1.25 (P1.4)
- new net: DA1.2 (COUT), VT1.2 (G1)
- new net: DA1.3 (DOUT), VT1.4 (G2)
- new net: C1.2, DA1.4 (VSS), GB01.2 (-), VT1.3 (S2)
- new net: C1.1, DA1.5 (BAT), R1.2
- new net: DA1.6 (V-), R2.1
- new net: VT1.5 (D2), VT1.6 (D2), VT1.7 (D1), VT1.8 (D1)
Other:
- moved on the sheet: C2, C3, C4, C5, C6, C7, DA2, DD1, L1, R3, R4, R5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
