File: PCB/Curse_PCB/Curse_PCB.sch (KiCad schematic (older format))
At the start: 26 parts

Commit message: docs
Parts:
- removed GB01: GB_BATTERY, Battery:BatteryHolder_Keystone_1042_1x18650, symbol KGL_Power:GB_BATTERY
- BQ1: renamed from ZQ1; value 32 kHz -> 32.768 kHz 03215C2; Тип (none) -> Кварцевый резонатор {Кварцевые резонаторы}
- C1, C3, C4: value 0.1 мкФ -> 0.1 мкФ-NP0-50В ±5% 0603; Тип (none) -> Конденсатор {Конденсаторы}
- C2, C6, C7: value 10 мкФ -> 10 мкФ-NP0-16В ±5% 0805; Тип (none) -> Конденсатор {Конденсаторы}
- C5: value 2200 пФ -> 2200 пФ-NP0-50В ±5% 0603; Тип (none) -> Конденсатор {Конденсаторы}
- DA1: value BQ29737 -> BQ29737 WSON-6; Тип (none) -> Микросхема {Микросхемы}
- DA2: value TPS63031 -> TPS63031 WSON-10; Тип (none) -> Микросхема {Микросхемы}
- DD1: value MSP430F2112 -> MSP430F2112IPW TSSOP-28; Тип (none) -> Микросхема {Микросхемы}
- L1: value 1,5 мкГн -> VLS252010CX-1R5M-1 1,5 мкГн 2010; Тип (none) -> Катушка индуктивности {Катушки индуктивности}
- R1: value 330 Ом -> 330 Ом ±5% 0603; Тип (none) -> Резистор {Резисторы}
- R2: value 2,2 кОм -> 2,2 кОм ±5% 0603; Тип (none) -> Резистор {Резисторы}
- R3, R4, R7, R8: value 10 кОм -> 10 кОм ±5% 0603; Тип (none) -> Резистор {Резисторы}
- R5: value 100 кОм -> 100 кОм ±5% 0603; Тип (none) -> Резистор {Резисторы}
- R6: value 47 кОм -> 47 кОм ±5% 0603; Тип (none) -> Резистор {Резисторы}
- SA1: value SA_SPST_NO -> PTS645VM58-2 LFS; Тип (none) -> Кнопка {Кнопки}
- VT1: value BUK9K5R1-30E -> BUK9K5R1-30E LFPAK56D; Тип (none) -> Транзистор {Транзисторы}
- XS1: value CONN_8 -> PBD-8; Тип (none) -> Разъём {Разъёмы}
- XS2, XS3: value CONN_4 -> PBS-4; Тип (none) -> Разъём {Разъёмы}
Changed lines of the file:
@@
 encoding utf-8
 Sheet 1 1
-Title "Схема электрическая\\nпринципиальная"
+Title "Плата обработки\\nСхема электрическая\\nпринципиальная"
 Date ""
 Rev ""
 Comp ""
-Comment1 "Плата обработки"
+Comment1 "Блок датчика"
 Comment2 ""
 Comment3 ""
@@
 U 1 1 616EA7AE
 P 8750 1650
-F 0 "R6" H 8750 1960 79  0000 C CNN
-F 1 "47 кОм" H 8750 1825 79  0000 C CNN
+F 0 "R6" H 8750 1842 79  0000 C CNN
+F 1 "47 кОм  ±5% 0603" H 8750 1825 79  0001 C CNN
 F 2 "Resistor_SMD:R_0603_1608Metric" H 8650 1675 60  0001 C CNN
 F 3 "" H 8775 1475 60  0001 C CNN
+F 4 "Резистор {Резисторы}" H 8750 1650 50  0001 C CNN "Тип"
 	1    8750 1650
 	1    0    0    -1
@@
 P 9100 4975
 F 0 "C4" H 9285 5043 79  0000 L CNN
-F 1 "0.1 мкФ" H 9285 4908 79  0000 L CNN
+F 1 "0.1 мкФ-NP0-50В ±5% 0603" H 9285 4908 79  0001 L CNN
 F 2 "Capacitor_SMD:C_0603_1608Metric" H 9025 4975 60  0001 C CNN
 F 3 "" H 9125 5075 60  0001 C CNN
+F 4 "Конденсатор {Конденсаторы}" H 9100 4975 50  0001 C CNN "Тип"
 	1    9100 4975
 	1    0    0    -1
@@
 P 11450 3200
 F 0 "DD1" H 11450 5045 79  0000 C CNN
-F 1 "MSP430F2112" H 11500 1250 79  0001 C CNN
+F 1 "MSP430F2112IPW TSSOP-28" H 11500 1250 79  0001 C CNN
 F 2 "Package_SO:TSSOP-28_4.4x9.7mm_P0.65mm" H 11500 1150 79  0001 C CNN
 F 3 "" H 11300 4400 98  0001 C CNN
+F 4 "Микросхема {Микросхемы}" H 11450 3200 50  0001 C CNN "Тип"
 	1    11450 3200
 	1    0    0    -1
 $EndComp
 $Comp
-L Device_GOST:ZQ_CRYSTAL ZQ1
+L Device_GOST:ZQ_CRYSTAL BQ1
 U 1 1 61700CB6
 P 9600 4150
-F 0 "ZQ1" V 9532 4296 79  0000 L CNN
-F 1 "32 kHz" V 9667 4296 79  0000 L CNN
+F 0 "BQ1" V 9532 4296 79  0000 L CNN
+F 1 "32.768 kHz 03215C2" V 9667 4296 79  0001 L CNN
 F 2 "" H 9500 4250 60  0001 C CNN
 F 3 "" H 9600 4350 60  0001 C CNN
+F 4 "Кварцевый резонатор {Кварцевые резонаторы}" V 9600 4150 50  0001 C CNN "Тип"
 	1    9600 4150
 	0    1    1    0
@@
 P 7250 8500
 F 0 "C3" H 7435 8568 79  0000 L CNN
-F 1 "0.1 мкФ" H 7435 8433 79  0000 L CNN
+F 1 "0.1 мкФ-NP0-50В ±5% 0603" H 7435 8433 79  0001 L CNN
 F 2 "Capacitor_SMD:C_0603_1608Metric" H 7175 8500 60  0001 C CNN
 F 3 "" H 7275 8600 60  0001 C CNN
+F 4 "Конденсатор {Конденсаторы}" H 7250 8500 50  0001 C CNN "Тип"
 	1    7250 8500
 	1    0    0    -1
@@
 P 9350 1975
 F 0 "C5" H 9535 2043 79  0000 L CNN
-F 1 "2200 пФ" H 9535 1908 79  0000 L CNN
+F 1 "2200 пФ-NP0-50В ±5% 0603" H 9535 1908 79  0001 L CNN
 F 2 "Capacitor_SMD:C_0603_1608Metric" H 9275 1975 60  0001 C CNN
 F 3 "" H 9375 2075 60  0001 C CNN
+F 4 "Конденсатор {Конденсаторы}" H 9350 1975 50  0001 C CNN "Тип"
 	1    9350 1975
 	1    0    0    -1
@@
 P 13450 2800
 F 0 "R7" V 13382 2907 79  0000 L CNN
-F 1 "10 кОм" V 13517 2907 79  0000 L CNN
+F 1 "10 кОм  ±5% 0603" V 13517 2907 79  0001 L CNN
 F 2 "Resistor_SMD:R_0603_1608Metric" H 13350 2825 60  0001 C CNN
 F 3 "" H 13475 2625 60  0001 C CNN
+F 4 "Резистор {Резисторы}" V 13450 2800 50  0001 C CNN "Тип"
 	1    13450 2800
 	0    1    1    0
@@
 P 14100 2800
 F 0 "R8" V 14032 2907 79  0000 L CNN
-F 1 "10 кОм" V 14167 2907 79  0000 L CNN
+F 1 "10 кОм  ±5% 0603" V 14167 2907 79  0001 L CNN
 F 2 "Resistor_SMD:R_0603_1608Metric" H 14000 2825 60  0001 C CNN
 F 3 "" H 14125 2625 60  0001 C CNN
+F 4 "Резистор {Резисторы}" V 14100 2800 50  0001 C CNN "Тип"
 	1    14100 2800
 	0    1    1    0
@@
 	13450 2450 13450 2200
 $Comp
-L KGL_Power:GB_BATTERY GB01
+L KGL_Power:GB_BATTERY #GB01
 U 1 1 617841BF
 P 1200 9350
-F 0 "GB01" V 1139 9535 70  0000 L CNN
-F 1 "GB_BATTERY" V 1260 9535 70  0000 L CNN
+F 0 "#GB01" V 1139 9535 70  0000 L CNN
+F 1 "GB_BATTERY" V 1260 9535 70  0001 L CNN
 F 2 "Battery:BatteryHolder_Keystone_1042_1x18650" H 1200 9350 70  0001 C CNN
 F 3 "" H 1200 9350 70  0001 C CNN
@@
 P 2100 3850
 F 0 "XS2" H 2090 4434 79  0000 C CNN
-F 1 "CONN_4" H 2100 3250 79  0001 C CNN
+F 1 "PBS-4" H 2100 3250 79  0001 C CNN
 F 2 "" H 2700 4450 79  0001 C CNN
 F 3 "" H 2700 3250 79  0001 C CNN
@@
 F 6 "AHT20_SCL" H 1893 3651 79  0000 C CNN "PIN3"
 F 7 "AHT20_SDA" H 1893 3450 79  0000 C CNN "PIN4"
+F 8 "Разъём {Разъёмы}" H 2100 3850 50  0001 C CNN "Тип"
 	1    2100 3850
 	1    0    0    -1
@@
 P 2100 2150
 F 0 "XS1" H 2090 3121 79  0000 C CNN
-F 1 "CONN_8" H 2100 1150 79  0001 C CNN
+F 1 "PBD-8" H 2100 1150 79  0001 C CNN
 F 2 "" H 2700 3150 79  0001 C CNN
 F 3 "" H 2700 1150 79  0001 C CNN
@@
 F 10 "ESP_REST" H 1893 1547 79  0000 C CNN "PIN7"
 F 11 "ESP_TX" H 1893 1346 79  0000 C CNN "PIN8"
+F 12 "Разъём {Разъёмы}" H 2100 2150 50  0001 C CNN "Тип"
 	1    2100 2150
 	1    0    0    -1
@@
 P 2100 5175
 F 0 "XS3" H 2090 5759 79  0000 C CNN
-F 1 "CONN_4" H 2100 4575 79  0001 C CNN
+F 1 "PBS-4" H 2100 4575 79  0001 C CNN
 F 2 "" H 2700 5775 79  0001 C CNN
 F 3 "" H 2700 4575 79  0001 C CNN
@@
 F 6 "DISP_SCL" H 1893 4976 79  0000 C CNN "PIN3"
 F 7 "DISP_SDA" H 1893 4775 79  0000 C CNN "PIN4"
+F 8 "Разъём {Разъёмы}" H 2100 5175 50  0001 C CNN "Тип"
 	1    2100 5175
 	1    0    0    -1
@@
 P 8850 7800
 F 0 "DA2" H 8850 8495 79  0000 C CNN
-F 1 "TPS63031" H 8800 7100 79  0001 C CNN
+F 1 "TPS63031 WSON-10" H 8800 7100 79  0001 C CNN
 F 2 "Package_SON:WSON-10-1EP_2.5x2.5mm_P0.5mm_EP1.2x2mm_ThermalVias" H 8850 8500 50  0001 C CNN
 F 3 "" H 8850 8500 50  0001 C CNN
+F 4 "Микросхема {Микросхемы}" H 8850 7800 50  0001 C CNN "Тип"
 	1    8850 7800
 	1    0    0    -1
@@
 U 1 1 6176016A
 P 8875 6600
-F 0 "L1" H 8875 6893 79  0000 C CNN
-F 1 "1,5 мкГн" H 8875 6758 79  0000 C CNN
+F 0 "L1" H 8875 6775 79  0000 C CNN
+F 1 "VLS252010CX-1R5M-1 1,5 мкГн 2010" H 8875 6758 79  0001 C CNN
 F 2 "" H 8775 6650 60  0001 C CNN
 F 3 "" H 8875 6750 60  0001 C CNN
+F 4 "Катушка индуктивности {Катушки индуктивности}" H 8875 6600 50  0001 C CNN "Тип"
 	1    8875 6600
 	1    0    0    -1
@@
 P 6375 7950
 F 0 "C2" H 6560 8018 79  0000 L CNN
-F 1 "10 мкФ" H 6560 7883 79  0000 L CNN
+F 1 "10 мкФ-NP0-16В ±5% 0805" H 6560 7883 79  0001 L CNN
 F 2 "Capacitor_SMD:C_0805_2012Metric" H 6300 7950 60  0001 C CNN
 F 3 "" H 6400 8050 60  0001 C CNN
+F 4 "Конденсатор {Конденсаторы}" H 6375 7950 50  0001 C CNN "Тип"
 	1    6375 7950
 	1    0    0    -1
@@
 P 10500 7950
 F 0 "C6" H 10685 8018 79  0000 L CNN
-F 1 "10 мкФ" H 10685 7883 79  0000 L CNN
+F 1 "10 мкФ-NP0-16В ±5% 0805" H 10685 7883 79  0001 L CNN
 F 2 "Capacitor_SMD:C_0805_2012Metric" H 10425 7950 60  0001 C CNN
 F 3 "" H 10525 8050 60  0001 C CNN
+F 4 "Конденсатор {Конденсаторы}" H 10500 7950 50  0001 C CNN "Тип"
 	1    10500 7950
 	1    0    0    -1
@@
 P 11400 7950
 F 0 "C7" H 11585 8018 79  0000 L CNN
-F 1 "10 мкФ" H 11585 7883 79  0000 L CNN
+F 1 "10 мкФ-NP0-16В ±5% 0805" H 11585 7883 79  0001 L CNN
 F 2 "Capacitor_SMD:C_0805_2012Metric" H 11325 7950 60  0001 C CNN
 F 3 "" H 11425 8050 60  0001 C CNN
+F 4 "Конденсатор {Конденсаторы}" H 11400 7950 50  0001 C CNN "Тип"
 	1    11400 7950
 	1    0    0    -1
@@
 P 5450 6650
 F 0 "R3" V 5382 6757 79  0000 L CNN
-F 1 "10 кОм" V 5517 6757 79  0000 L CNN
+F 1 "10 кОм  ±5% 0603" V 5517 6757 79  0001 L CNN
 F 2 "Resistor_SMD:R_0603_1608Metric" H 5350 6675 60  0001 C CNN
 F 3 "" H 5475 6475 60  0001 C CNN
+F 4 "Резистор {Резисторы}" V 5450 6650 50  0001 C CNN "Тип"
 	1    5450 6650
 	0    1    1    0
@@
 U 1 1 617CC1AA
 P 6050 6100
-F 0 "R4" H 6050 6410 79  0000 C CNN
-F 1 "10 кОм" H 6050 6275 79  0000 C CNN
+F 0 "R4" H 6050 6291 79  0000 C CNN
+F 1 "10 кОм  ±5% 0603" H 6050 6275 79  0001 C CNN
 F 2 "Resistor_SMD:R_0603_1608Metric" H 5950 6125 60  0001 C CNN
 F 3 "" H 6075 5925 60  0001 C CNN
+F 4 "Резистор {Резисторы}" H 6050 6100 50  0001 C CNN "Тип"
 	1    6050 6100
 	1    0    0    -1
@@
 P 6950 2850
 F 0 "SA1" H 6950 3081 79  0000 C CNN
-F 1 "SA_SPST_NO" H 6950 2750 79  0001 C CNN
+F 1 "PTS645VM58-2 LFS" H 6950 2750 79  0001 C CNN
 F 2 "Button_Switch_THT:SW_Tactile_SPST_Angled_PTS645Vx58-2LFS" H 6850 2950 98  0001 C CNN
 F 3 "" H 6950 3050 98  0001 C CNN
+F 4 "Кнопка {Кнопки}" H 6950 2850 50  0001 C CNN "Тип"
 	1    6950 2850
 	-1   0    0    -1
@@
 P 7900 3350
 F 0 "R5" V 7832 3457 79  0000 L CNN
-F 1 "100 кОм" V 7967 3457 79  0000 L CNN
+F 1 "100 кОм  ±5% 0603" V 7967 3457 79  0001 L CNN
 F 2 "" H 7800 3375 60  0001 C CNN
 F 3 "" H 7925 3175 60  0001 C CNN
+F 4 "Резистор {Резисторы}" V 7900 3350 50  0001 C CNN "Тип"
 	1    7900 3350
 	0    1    1    0
@@
 P 4400 8900
 F 0 "DA1" H 4400 9395 79  0000 C CNN
-F 1 "BQ29737" H 4400 8400 79  0001 C CNN
+F 1 "BQ29737 WSON-6" H 4400 8400 79  0001 C CNN
 F 2 "Package_SON:WSON-6_1.5x1.5mm_P0.5mm" H 4400 9400 50  0001 C CNN
 F 3 "" H 4400 9400 50  0001 C CNN
+F 4 "Микросхема {Микросхемы}" H 4400 8900 50  0001 C CNN "Тип"
 	1    4400 8900
 	-1   0    0    -1
@@
 P 2750 9350
 F 0 "C1" H 2935 9418 79  0000 L CNN
-F 1 "0.1 мкФ" H 2935 9283 79  0000 L CNN
+F 1 "0.1 мкФ-NP0-50В ±5% 0603" H 2935 9283 79  0001 L CNN
 F 2 "Capacitor_SMD:C_0603_1608Metric" H 2675 9350 60  0001 C CNN
 F 3 "" H 2775 9450 60  0001 C CNN
+F 4 "Конденсатор {Конденсаторы}" H 2750 9350 50  0001 C CNN "Тип"
 	1    2750 9350
 	1    0    0    -1
@@
 P 2750 8250
 F 0 "R1" V 2682 8357 79  0000 L CNN
-F 1 "330 Ом" V 2817 8357 79  0000 L CNN
+F 1 "330 Ом ±5% 0603" V 2817 8357 79  0001 L CNN
 F 2 "Resistor_SMD:R_0603_1608Metric" H 2650 8275 60  0001 C CNN
 F 3 "" H 2775 8075 60  0001 C CNN
+F 4 "Резистор {Резисторы}" V 2750 8250 50  0001 C CNN "Тип"
 	1    2750 8250
 	0    1    1    0
@@
 P 7550 10100
 F 0 "VT1" H 7550 10695 79  0000 C CNN
-F 1 "BUK9K5R1-30E" H 7550 9500 79  0001 C CNN
+F 1 "BUK9K5R1-30E LFPAK56D" H 7550 9500 79  0001 C CNN
 F 2 "Package_TO_SOT_SMD:LFPAK56D" H 7550 10700 50  0001 C CNN
 F 3 "" H 7550 10700 50  0001 C CNN
+F 4 "Транзистор {Транзисторы}" H 7550 10100 50  0001 C CNN "Тип"
 	1    7550 10100
 	1    0    0    -1
@@
 U 1 1 6172E895
 P 4375 8100
-F 0 "R2" H 4375 8410 79  0000 C CNN
-F 1 "2,2 кОм" H 4375 8275 79  0000 C CNN
+F 0 "R2" H 4375 8275 79  0000 C CNN
+F 1 "2,2 кОм  ±5% 0603" H 4375 8275 79  0001 C CNN
 F 2 "Resistor_SMD:R_0603_1608Metric" H 4275 8125 60  0001 C CNN
 F 3 "" H 4400 7925 60  0001 C CNN
+F 4 "Резистор {Резисторы}" H 4375 8100 50  0001 C CNN "Тип"
 	1    4375 8100
 	1    0    0    -1

Commit message: pcb
Parts:
- BQ1: footprint (none) -> Crystal:Crystal_SMD_3215-2Pin_3.2x1.5mm
- DA1: symbol My_Lib_GOST:BQ297xx -> Curse_PCB-rescue:BQ297xx-My_Lib_GOST
- DA2: symbol My_Lib_GOST:TPS6303x -> Curse_PCB-rescue:TPS6303x-My_Lib_GOST
- DD1: symbol My_Lib_GOST:MSP430F21x2 -> Curse_PCB-rescue:MSP430F21x2-My_Lib_GOST
- L1: footprint (none) -> myLib_LCC:VLS252012CX
- R5: footprint (none) -> Resistor_SMD:R_0603_1608Metric
- VT1: footprint Package_TO_SOT_SMD:LFPAK56D -> myLib_LCC:LFPAK56D; symbol My_Lib_GOST:BUK9K5R1-30E -> Curse_PCB-rescue:BUK9K5R1-30E-My_Lib_GOST
- XS1: footprint (none) -> Connector_PinSocket_2.54mm:PinSocket_2x04_P2.54mm_Vertical_SMD
- XS2, XS3: footprint (none) -> Connector_PinSocket_2.54mm:PinSocket_1x04_P2.54mm_Vertical
Changed lines of the file:
@@
 $EndComp
 $Comp
-L My_Lib_GOST:MSP430F21x2 DD1
+L Curse_PCB-rescue:MSP430F21x2-My_Lib_GOST DD1
 U 1 1 616F7B6C
 P 11450 3200
@@
 F 0 "BQ1" V 9532 4296 79  0000 L CNN
 F 1 "32.768 kHz 03215C2" V 9667 4296 79  0001 L CNN
-F 2 "" H 9500 4250 60  0001 C CNN
+F 2 "Crystal:Crystal_SMD_3215-2Pin_3.2x1.5mm" H 9500 4250 60  0001 C CNN
 F 3 "" H 9600 4350 60  0001 C CNN
 F 4 "Кварцевый резонатор {Кварцевые резонаторы}" V 9600 4150 50  0001 C CNN "Тип"
@@
 	9100 4650 10350 4650
 $Comp
-L power_GOST:+3.3V #PWR014
+L Curse_PCB-rescue:+3.3V-power_GOST #PWR014
 U 1 1 6170F574
 P 8600 4150
@@
 	9350 1775 9350 1650
 $Comp
-L power_GOST:+3.3V #PWR012
+L Curse_PCB-rescue:+3.3V-power_GOST #PWR012
 U 1 1 6171A6D2
 P 7900 1150
@@
 	14100 3450 14600 3450
 $Comp
-L power_GOST:+3.3V #PWR022
+L Curse_PCB-rescue:+3.3V-power_GOST #PWR022
 U 1 1 617452FA
 P 13450 2200
@@
 $EndComp
 $Comp
-L power_GOST:+3.3V #PWR023
+L Curse_PCB-rescue:+3.3V-power_GOST #PWR023
 U 1 1 61747566
 P 14100 2200
@@
 	13450 2450 13450 2200
 $Comp
-L KGL_Power:GB_BATTERY #GB01
+L Curse_PCB-rescue:GB_BATTERY-KGL_Power #GB01
 U 1 1 617841BF
 P 1200 9350
 F 0 "#GB01" V 1139 9535 70  0000 L CNN
-F 1 "GB_BATTERY" V 1260 9535 70  0001 L CNN
+F 1 "GB_BATTERY-KGL_Power" V 1260 9535 70  0001 L CNN
 F 2 "Battery:BatteryHolder_Keystone_1042_1x18650" H 1200 9350 70  0001 C CNN
 F 3 "" H 1200 9350 70  0001 C CNN
@@
 F 0 "XS2" H 2090 4434 79  0000 C CNN
 F 1 "PBS-4" H 2100 3250 79  0001 C CNN
-F 2 "" H 2700 4450 79  0001 C CNN
+F 2 "Connector_PinSocket_2.54mm:PinSocket_1x04_P2.54mm_Vertical" H 2700 4450 79  0001 C CNN
 F 3 "" H 2700 3250 79  0001 C CNN
 F 4 "AHT20_VCC" H 1893 4049 79  0000 C CNN "PIN1"
@@
 F 0 "XS1" H 2090 3121 79  0000 C CNN
 F 1 "PBD-8" H 2100 1150 79  0001 C CNN
-F 2 "" H 2700 3150 79  0001 C CNN
+F 2 "Connector_PinSocket_2.54mm:PinSocket_2x04_P2.54mm_Vertical_SMD" H 2700 3150 79  0001 C CNN
 F 3 "" H 2700 1150 79  0001 C CNN
 F 4 "ESP_GND" H 1893 2749 79  0000 C CNN "PIN1"
@@
 $EndComp
 $Comp
-L power_GOST:+3.3V #PWR02
+L Curse_PCB-rescue:+3.3V-power_GOST #PWR02
 U 1 1 61735273
 P 3700 2225
@@
 F 0 "XS3" H 2090 5759 79  0000 C CNN
 F 1 "PBS-4" H 2100 4575 79  0001 C CNN
-F 2 "" H 2700 5775 79  0001 C CNN
+F 2 "Connector_PinSocket_2.54mm:PinSocket_1x04_P2.54mm_Vertical" H 2700 5775 79  0001 C CNN
 F 3 "" H 2700 4575 79  0001 C CNN
 F 4 "DISP_GND" H 1893 5374 79  0000 C CNN "PIN1"
@@
 $EndComp
 $Comp
-L power_GOST:+3.3V #PWR03
+L Curse_PCB-rescue:+3.3V-power_GOST #PWR03
 U 1 1 61746EB1
 P 3700 3525
@@
 	3700 3650 3700 3525
 $Comp
-L power_GOST:+3.3V #PWR05
+L Curse_PCB-rescue:+3.3V-power_GOST #PWR05
 U 1 1 61747917
 P 3700 5050
@@
 	2900 3850 3700 3850
 $Comp
-L My_Lib_GOST:TPS6303x DA2
+L Curse_PCB-rescue:TPS6303x-My_Lib_GOST DA2
 U 1 1 6175C4E8
 P 8850 7800
@@
 F 0 "L1" H 8875 6775 79  0000 C CNN
 F 1 "VLS252010CX-1R5M-1 1,5 мкГн 2010" H 8875 6758 79  0001 C CNN
-F 2 "" H 8775 6650 60  0001 C CNN
+F 2 "myLib_LCC:VLS252012CX" H 8775 6650 60  0001 C CNN
 F 3 "" H 8875 6750 60  0001 C CNN
 F 4 "Катушка индуктивности {Катушки индуктивности}" H 8875 6600 50  0001 C CNN "Тип"
@@
 	10000 7600 10500 7600
 $Comp
-L power_GOST:+3.3V #PWR021
+L Curse_PCB-rescue:+3.3V-power_GOST #PWR021
 U 1 1 617A17C2
 P 11750 7100
@@
 $EndComp
 $Comp
-L power_GOST:+3.3V #PWR09
+L Curse_PCB-rescue:+3.3V-power_GOST #PWR09
 U 1 1 618650BF
 P 6200 2600
@@
 F 0 "R5" V 7832 3457 79  0000 L CNN
 F 1 "100 кОм  ±5% 0603" V 7967 3457 79  0001 L CNN
-F 2 "" H 7800 3375 60  0001 C CNN
+F 2 "Resistor_SMD:R_0603_1608Metric" H 7800 3375 60  0001 C CNN
 F 3 "" H 7925 3175 60  0001 C CNN
 F 4 "Резистор {Резисторы}" V 7900 3350 50  0001 C CNN "Тип"
@@
 	7900 3000 7900 2850
 $Comp
-L My_Lib_GOST:BQ297xx DA1
+L Curse_PCB-rescue:BQ297xx-My_Lib_GOST DA1
 U 1 1 61707952
 P 4400 8900
@@
 Connection ~ 6375 7600
 $Comp
-L My_Lib_GOST:BUK9K5R1-30E VT1
+L Curse_PCB-rescue:BUK9K5R1-30E-My_Lib_GOST VT1
 U 1 1 6170DBC2
 P 7550 10100
 F 0 "VT1" H 7550 10695 79  0000 C CNN
 F 1 "BUK9K5R1-30E LFPAK56D" H 7550 9500 79  0001 C CNN
-F 2 "Package_TO_SOT_SMD:LFPAK56D" H 7550 10700 50  0001 C CNN
+F 2 "myLib_LCC:LFPAK56D" H 7550 10700 50  0001 C CNN
 F 3 "" H 7550 10700 50  0001 C CNN
 F 4 "Транзистор {Транзисторы}" H 7550 10100 50  0001 C CNN "Тип"

Commit message: sch + pcb
Parts:
- added GB1: Battery_Cell, Battery:BatteryHolder_Keystone_2462_2xAA, symbol Device:Battery_Cell
- added R10, R12, R13, R14, R15, R9: 510 Ом ±5% 0603, Resistor_SMD:R_0603_1608Metric, symbol Device_GOST:R
- added SA?: PTS645VM58-2 LFS, Button_Switch_THT:SW_Tactile_SPST_Angled_PTS645Vx58-2LFS, symbol Device_GOST:SA_SPST_NO
- added VT2: Si2307BDS, Package_TO_SOT_SMD:SOT-23, symbol Device_GOST:VT_PMOS_GSD
- added XS4: Type_C_Amphenol_124018802112A, symbol Connector_Specialized_GOST:Type_C_Amphenol_124018802112A
Connections:
- net ESP_CH_PD: now also R15.1; no longer DD1.27 (P1.6)
- net ESP_IO0: now also R14.1; no longer DD1.25 (P1.4)
- net ESP_IO2: now also R12.1; no longer DD1.26 (P1.5)
- net ESP_REST: now also R13.1; no longer DD1.28 (P1.7)
- net UART_RX: now also R10.2; no longer DD1.16 (P3.5)
- net UART_TX: now also R9.2; no longer DD1.15 (P3.4)
- net at C1.2, DA1.4 (VSS), VT1.3 (S2): now also GB1.2 (-), VT2.1 (G)
- net at C2.1, DA2.5 (VIN), R1.1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: now also VT2.2 (S)
- new net: DD1.15 (P3.4), R9.1
- new net: DD1.16 (P3.5), R10.1
- new net: DD1.25 (P1.4), R14.2
- new net: DD1.26 (P1.5), R12.2
- new net: DD1.27 (P1.6), R15.2
- new net: DD1.28 (P1.7), R13.2
- new net: GB1.1 (+), VT2.3 (D)
Other:
- note added: "Внешние нагрузочные \nёмкости не требуются, \nтак как контроллер \nимеет встроенные"
- note added: "Для предотвращения \nвыхода контроллра из \nстроя напряжение \nна АЦП подаётся \nчерез делитель, который \nделит напряжение пополам"
- note added: "Защита аккумулятора\nот перезаряда и переразряда"
- note added: "Защита выводов микосхемы"
- note added: "Защита от\nпереполюсовки"
- note added: "Подключение вывода ~RST~ согласно документации"
- note added: "Подключение питания \nмикросхемы согласно \nдокументации"
- note added: "Подключение преобразователя\nсогласно документации"
- moved on the sheet: R5, SA1
