File: PCB/Curse_PCB/Curse_PCB.sch (KiCad schematic (older format))
At the start: 35 parts

Commit message: upd
Parts:
- removed XS4: Type_C_Amphenol_124018802112A, symbol Connector_Specialized_GOST:Type_C_Amphenol_124018802112A
- added C2: 1 мкФ-NP0-16В ±5% 0805, Capacitor_SMD:C_0805_2012Metric, symbol Device_GOST:C
- added DA2: BQ21040, Package_TO_SOT_SMD:SOT-23-6, symbol Power_Management_GOST:BQ21040
- added HL1: HL_LED, LED_SMD:LED_0603_1608Metric, symbol Device_GOST:HL_LED
- added R12: 47 кОм ±5% 0603, Resistor_SMD:R_0603_1608Metric, symbol Device_GOST:R
- added R2: 1,0 кОм ±1% 0603, Resistor_SMD:R_0603_1608Metric, symbol Device_GOST:R
- added R4: 10 кОм ±5% 0603, Resistor_SMD:R_0603_1608Metric, symbol Device_GOST:R
- added R6: 1,5 кОм ±5% 0603, Resistor_SMD:R_0603_1608Metric, symbol Device_GOST:R
- added XS4: 5.5x2.1, Connector_BarrelJack:BarrelJack_CUI_PJ-063AH_Horizontal, symbol Connector_Generic_GOST:CONN_2
- GB1: Тип (none) -> Прочее
- R9: renamed from R6; value 47 кОм ±5% 0603 -> 100 Ом ±5% 0603
- VT1: renamed from VT2; Тип (none) -> Транзистор {Транзисторы}
- gave numbers to parts that had none: 1
- renumbered C2 to C3, C3 to C4, C4 to C5, C5 to C6, C6 to C7, C7 to C8, DA2 to DA3, R12 to R10, R13 to R11, R14 to R13, R15 to R14, R7 to R15, R9 to R16, R8 to R17, R10 to R18, R2 to R3, R3 to R5, R4 to R7, R5 to R8, VT1 to VT2
Connections:
- net +3.3V: now also R12.1; no longer R9.1
- net EXP: now also R9.1, C2.2, DA2.5 (GND), R2.2, R4.2, XS4.2
- net at C6.1, DD1.7 (~RST): now also SA2.1, R12.2; no longer R9.2
- net at C3.1, DA3.5 (VIN), R1.1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: now also DA2.2 (VOUT), R6.2
- net at SA2.2: now also R9.2
- new net: C2.1, DA2.6 (VIN), XS4.1
- new net: DA2.1 (TS), R4.1
- new net: DA2.3 (~CHG), HL1.1 (K)
- new net: DA2.4 (ISET), R2.1
- new net: HL1.2 (A), R6.1
Other:
- note added: "RESET"
- note added: "Подключение кнопки"
- note added: "Разъём и микросхема для зарядки аккумулятора"
- note added: "Разём для подключения ESP"
- note added: "Разём для подключения OLED-дисплея"
- note added: "Разём для подключения датчика AHT20"
- moved on the sheet: BQ1, C1, C3, C4, C5, C6, C7, C8, DA1, DA3, DD1, GB1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
