File: PCB/Curse_PCB/Curse_PCB.kicad_pcb (KiCad board)
At the start: 2 copper layers, 23.4 x 24.9 mm, 14 parts

Commit message: SCH + PCB
Parts:
- removed TP1: 32.768 kHz TP, TestPoint:TestPoint_THTPad_D1.0mm_Drill0.5mm
- added XP4: I2C_SENSOR_CONN, Connector_PinHeader_2.54mm:PinHeader_1x04_P2.54mm_Vertical, F.Cu at (77.9, 55.9)
- added XP7: ADC1_CONN, Connector_PinHeader_2.54mm:PinHeader_1x03_P2.54mm_Vertical, F.Cu at (58.8, 56.8)
- BQ1: footprint Crystal:Crystal_DS26_D2.0mm_L6.0mm_Horizontal -> Crystal:Crystal_SMD_3215-2Pin_3.2x1.5mm
- R1, R2: value 47K -> 10K
- moved XP6 18.4 mm to (58.8, 65.5), turned to 90 degrees
- moved XP1 17.2 mm to (60.8, 44.4), turned to 270 degrees
- moved XP2 9.05 mm to (77.9, 44.6)
- moved XP5 4.86 mm to (58.8, 48.0)
- moved R4 2.50 mm to (62.2, 53.2), turned to 90 degrees
- moved R1 2.49 mm to (72.5, 63.5)
- moved R2 2.29 mm to (74.1, 60.2)
- moved C1 1.51 mm to (62.0, 59.1), turned to 90 degrees
- moved BQ1 1.40 mm to (64.9, 61.9), turned to 0 degrees
Connections:
- net Net-(DD1-Pad12) renamed /SDA
- net Net-(DD1-Pad13) renamed /SCL
- DD1 pad 17: Net-(DD1-Pad17) -> /ADC_CH6
- DD1 pad 18: Net-(DD1-Pad18) -> /ADC_CH7
- XP5 pad 2: Net-(XP5-Pad2) -> /ADC_CH6
Routing:
- net /ADC_CH7: track 0.00 -> 14.7 mm
- net /SDA: track 8.21 -> 22.8 mm
- net /ADC_CH6: track 0.00 -> 13.9 mm
- net /SCL: track 7.83 -> 20.5 mm
- net /BTN0: track 10.0 -> 20.8 mm
- net +3V3: track 74.1 -> 69.2 mm, vias 0 -> 3
- net Net-(BQ1-Pad2): track 2.44 -> 5.24 mm
- net Net-(DD1-Pad8): track 1.96 -> 0.00 mm
- net Net-(BQ1-Pad1): track 4.61 -> 3.69 mm
- net GND: vias 0 -> 2
- added copper zone on B.Cu, net +3V3
Other:
- board size 23.4 x 24.9 mm -> 25.4 x 24.9 mm

Commit message: АЦП
Parts:
- removed XP7: ADC1_CONN, Connector_PinHeader_2.54mm:PinHeader_1x03_P2.54mm_Vertical
- added R5: 10K, Resistor_SMD:R_0603_1608Metric, F.Cu at (64.5, 50.0)
- added R6: 10K, Resistor_SMD:R_0603_1608Metric, F.Cu at (67.1, 50.9)
- XP1: footprint Connector_PinHeader_2.54mm:PinHeader_1x02_P2.54mm_Vertical -> Connector_PinHeader_2.54mm:PinHeader_1x03_P2.54mm_Vertical
- moved XP5 5.87 mm to (59.0, 53.9)
- moved XP1 1.94 mm to (59.0, 45.0), turned to 0 degrees
- moved R4 1.15 mm to (62.0, 54.3), turned to 270 degrees
Connections:
- DD1 pad 17: /ADC_CH6 -> Net-(DD1-Pad17)
- DD1 pad 18: /ADC_CH7 -> Net-(DD1-Pad18)
- DD1 pad 20: Net-(DD1-Pad20) -> /BAT_ADC
- DD1 pad 3: Net-(DD1-Pad3) -> /DS18B20
- XP5 pad 2: /ADC_CH6 -> /DS18B20
Routing:
- net /ADC_CH7: track 14.7 -> 0.00 mm
- net /ADC_CH6: track 13.9 -> 0.00 mm
- net +3V3: track 69.2 -> 79.1 mm
- net /DS18B20: track 0.00 -> 7.95 mm
- net Net-(R5-Pad1): track 0.00 -> 7.62 mm
- net /BTN0: track 20.8 -> 24.5 mm
- net /BAT_ADC: track 0.00 -> 2.91 mm
- net GND: track 1.24 -> 3.54 mm
- removed copper zone on B.Cu, net +3V3

Commit message: LDO
Parts:
- added C3: 10 uF, Capacitor_SMD:C_0603_1608Metric, B.Cu at (60.4, 61.3)
- added C4: 10 uF, Capacitor_SMD:C_0603_1608Metric, B.Cu at (62.7, 53.9)
- added DA1: AMS1117-3.3, Package_TO_SOT_SMD:SOT-223-3_TabPin2, B.Cu at (66.2, 62.8)
- moved XP6 21.2 mm to (57.5, 44.3)
- moved R5 17.4 mm to (71.1, 66.1), turned to 0 degrees
- moved XP1 15.6 mm to (57.5, 60.5)
- moved R6 13.3 mm to (70.3, 63.8), turned to 90 degrees
- moved XP5 5.93 mm to (57.5, 48.2)
- moved R4 5.92 mm to (66.8, 50.8), turned to 0 degrees
- moved R1 1.63 mm to (74.1, 63.5)
- moved C2 1.56 mm to (67.2, 64.6)
- moved R3 0.82 mm to (67.9, 62.2), turned to 90 degrees
- moved BQ1 0.48 mm to (64.5, 62.1), turned to 270 degrees
Connections:
- DD1 pad 20: /BAT_ADC -> Net-(DD1-Pad20)
- DD1 pad 8: Net-(DD1-Pad8) -> /BAT_ADC
- XP1 pad 1: +3V3 -> +5V
Routing:
- net +3V3: track 79.1 -> 33.9 mm, vias 3 -> 1
- net /BTN0: track 24.5 -> 13.3 mm
- net Net-(R5-Pad1): track 7.62 -> 14.6 mm
- net +5V: track 0.00 -> 5.57 mm
- net /DS18B20: track 7.95 -> 12.6 mm
- net Net-(BQ1-Pad1): track 3.69 -> 5.86 mm
- net /BAT_ADC: track 2.91 -> 5.03 mm
- net Net-(BQ1-Pad2): track 5.24 -> 3.47 mm
- net Net-(C2-Pad1): track 5.56 -> 6.51 mm

Commit message: pcb
Parts:
- removed XP1: POWER_CONN, Connector_PinHeader_2.54mm:PinHeader_1x03_P2.54mm_Vertical
- removed XP2: DISP_CONN, Connector_PinHeader_2.54mm:PinHeader_1x04_P2.54mm_Vertical
- removed XP3: ESP_CONN, Connector_PinSocket_2.54mm:PinSocket_2x04_P2.54mm_Vertical
- removed XP4: I2C_SENSOR_CONN, Connector_PinHeader_2.54mm:PinHeader_1x04_P2.54mm_Vertical
- removed XP5: ADC0_CONN, Connector_PinHeader_2.54mm:PinHeader_1x03_P2.54mm_Vertical
- removed XP6: BTN_CONN, Connector_PinHeader_2.54mm:PinHeader_1x02_P2.54mm_Vertical
- added C5: 2200 пФ-NP0-50В ±5% 0603, Capacitor_SMD:C_0603_1608Metric, F.Cu at (79.4, 58.6)
- added C6: 10 мкФ-NP0-16В ±5% 0805, Capacitor_SMD:C_0805_2012Metric, F.Cu at (67.2, 62.0)
- added C7: 10 мкФ-NP0-16В ±5% 0805, Capacitor_SMD:C_0805_2012Metric, F.Cu at (80.7, 55.5)
- added DA2: TPS63031 WSON-10, Package_SON:WSON-10-1EP_2.5x2.5mm_P0.5mm_EP1.2x2mm_ThermalVias, F.Cu at (86.7, 55.1)
- added L1: VLS252010CX-1R5M-1 1,5 мкГн 2010, myLib_LCC:VLS252012CX, F.Cu at (95.7, 55.7)
- added R7: 10 кОм ±5% 0603, Resistor_SMD:R_0603_1608Metric, F.Cu at (100.9, 54.2)
- added R8: 10 кОм ±5% 0603, Resistor_SMD:R_0603_1608Metric, F.Cu at (92.0, 60.2)
- added SA1: PTS645VM58-2 LFS, Button_Switch_THT:SW_Tactile_SPST_Angled_PTS645Vx58-2LFS, F.Cu at (87.3, 48.1)
- added VT1: BUK9K5R1-30E LFPAK56D, myLib_LCC:LFPAK56D, F.Cu at (69.2, 57.2)
- added XS1: PBD-8, Connector_PinSocket_2.54mm:PinSocket_2x04_P2.54mm_Vertical_SMD, F.Cu at (79.3, 47.8)
- added XS2: PBS-4, Connector_PinSocket_2.54mm:PinSocket_1x04_P2.54mm_Vertical, F.Cu at (71.9, 44.0)
- added XS3: PBS-4, Connector_PinSocket_2.54mm:PinSocket_1x04_P2.54mm_Vertical, F.Cu at (67.3, 44.0)
- BQ1: value Crystal -> 32.768 kHz 03215C2
- C1: value 0.1 uF -> 0.1 мкФ-NP0-50В ±5% 0603
- C2: value 2200 pF -> 10 мкФ-NP0-16В ±5% 0805; footprint Capacitor_SMD:C_0603_1608Metric -> Capacitor_SMD:C_0805_2012Metric
- C3, C4: value 10 uF -> 0.1 мкФ-NP0-50В ±5% 0603; moved to F.Cu
- DA1: value AMS1117-3.3 -> BQ29737 WSON-6; footprint Package_TO_SOT_SMD:SOT-223-3_TabPin2 -> Package_SON:WSON-6_1.5x1.5mm_P0.5mm; moved to F.Cu
- DD1: value MSP430F2112IPW -> MSP430F2112IPW TSSOP-28
- R1: value 10K -> 330 Ом ±5% 0603
- R2: value 10K -> 2,2 кОм ±5% 0603
- R3, R4: value 47K -> 10 кОм ±5% 0603
- R5: value 10K -> 100 кОм ±5% 0603
- R6: value 10K -> 47 кОм ±5% 0603
- moved DA1 34.9 mm to (100.7, 57.0)
- moved DD1 32.2 mm to (99.3, 47.3), turned to 0 degrees
- moved R4 22.0 mm to (87.4, 58.4)
- moved R5 22.0 mm to (91.4, 57.7)
- moved C1 21.4 mm to (83.4, 58.4), turned to 0 degrees
- moved R1 19.3 mm to (91.1, 54.3), turned to 0 degrees
- moved R6 17.9 mm to (87.9, 60.9), turned to 0 degrees
- moved R3 16.1 mm to (83.9, 60.9), turned to 0 degrees
- moved C3 15.2 mm to (75.4, 58.6), turned to 0 degrees
- moved C4 15.0 mm to (75.9, 61.1)
- moved BQ1 13.2 mm to (75.9, 55.6), turned to 0 degrees
- moved R2 5.89 mm to (79.9, 61.1), turned to 0 degrees
- moved C2 5.17 mm to (71.7, 62.0)
Connections:
- C1 pad 1: +3V3 -> Net-(C1-Pad1)
- C1 pad 2: GND -> Net-(C1-Pad2)
- C2 pad 2: GND -> EXP
- C3 pad 1: +5V -> Net-(C3-Pad1)
- C3 pad 2: GND -> EXP
- C4 pad 1: +3V3 -> +3.3V
- C4 pad 2: GND -> EXP
- DA1 pad 1: GND -> Net-(DA1-Pad1)
- DA1 pad 2: +3V3 -> Net-(DA1-Pad2)
- DA1 pad 3: +5V -> Net-(DA1-Pad3)
- DD1 pad 2: +3V3 -> +3.3V
- DD1 pad 25: /BTN0 -> /ESP_IO0
- DD1 pad 26: Net-(DD1-Pad26) -> /ESP_IO2
- DD1 pad 27: Net-(DD1-Pad27) -> /ESP_CH_PD
- DD1 pad 28: Net-(DD1-Pad28) -> /ESP_REST
- DD1 pad 3: /DS18B20 -> Net-(DD1-Pad3)
- DD1 pad 4: GND -> EXP
- DD1 pad 7: Net-(C2-Pad1) -> Net-(C5-Pad1)
- R1 pad 1: +3V3 -> Net-(C2-Pad1)
- R1 pad 2: /SDA -> Net-(C1-Pad1)
- R2 pad 1: +3V3 -> Net-(DA1-Pad6)
- R2 pad 2: /SCL -> EXP
- R3 pad 1: +3V3 -> Net-(C2-Pad1)
- R3 pad 2: Net-(C2-Pad1) -> EXP
- R4 pad 1: /BTN0 -> Net-(C2-Pad1)
- R4 pad 2: GND -> /BAT_ADC
- R5 pad 1: Net-(R5-Pad1) -> Net-(DD1-Pad24)
- R5 pad 2: GND -> EXP
- R6 pad 1: Net-(R5-Pad1) -> +3.3V
- R6 pad 2: /BAT_ADC -> Net-(C5-Pad1)
Routing:
- net +3V3: track 33.9 -> 0.00 mm, vias 1 -> 0
- net /SDA: track 22.8 -> 0.00 mm
- net /SCL: track 20.5 -> 0.00 mm
- net Net-(R5-Pad1): track 14.6 -> 0.00 mm
- net /UART_RX: track 13.6 -> 0.00 mm
- net /BTN0: track 13.3 -> 0.00 mm
- net /DS18B20: track 12.6 -> 0.00 mm
- net /UART_TX: track 10.9 -> 0.00 mm
- net Net-(C2-Pad1): track 6.51 -> 0.00 mm
- net Net-(BQ1-Pad1): track 5.86 -> 0.00 mm
- net +5V: track 5.57 -> 0.00 mm
- net /BAT_ADC: track 5.03 -> 0.00 mm
- net GND: track 3.54 -> 0.00 mm, vias 2 -> 0
- net Net-(BQ1-Pad2): track 3.47 -> 0.00 mm
- removed copper zone on B.Cu, net GND
- removed copper zone on F.Cu, net GND
Other:
- board outline removed

Commit message: sch + pcb
Parts:
- added GB1: Battery_Cell, Battery:BatteryHolder_Keystone_2462_2xAA, B.Cu at (111.0, 43.0)
- added R10: 510 Ом ±5% 0603, Resistor_SMD:R_0603_1608Metric, F.Cu at (115.8, 102.5)
- added R12: 510 Ом ±5% 0603, Resistor_SMD:R_0603_1608Metric, F.Cu at (113.9, 87.8)
- added R13: 510 Ом ±5% 0603, Resistor_SMD:R_0603_1608Metric, F.Cu at (113.8, 85.6)
- added R14: 510 Ом ±5% 0603, Resistor_SMD:R_0603_1608Metric, F.Cu at (118.0, 82.1)
- added R15: 510 Ом ±5% 0603, Resistor_SMD:R_0603_1608Metric, F.Cu at (117.2, 87.2)
- added R9: 510 Ом ±5% 0603, Resistor_SMD:R_0603_1608Metric, F.Cu at (111.7, 102.5)
- added VT2: Si2307BDS, Package_TO_SOT_SMD:SOT-23, F.Cu at (94.0, 82.5)
- moved XS1 53.8 mm to (133.0, 50.0), turned to 90 degrees
- moved R2 47.3 mm to (76.7, 108.2)
- moved R8 47.3 mm to (88.7, 107.4)
- moved R5 47.3 mm to (88.2, 104.9)
- moved R7 45.0 mm to (96.5, 99.0)
- moved DD1 43.9 mm to (106.0, 90.7)
- moved BQ1 40.8 mm to (98.7, 89.4), turned to 270 degrees
- moved VT1 39.9 mm to (108.4, 64.7)
- moved C5 39.8 mm to (96.9, 94.3), turned to 270 degrees
- moved C4 35.8 mm to (101.2, 86.4), turned to 90 degrees
- moved R6 33.3 mm to (94.5, 93.6)
- moved C6 31.6 mm to (98.1, 55.1), turned to 180 degrees
- moved C2 28.3 mm to (100.0, 60.3)
- moved C3 27.6 mm to (103.0, 59.5), turned to 270 degrees
- moved C1 20.3 mm to (103.0, 63.9)
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Connections:
- DD1 pad 15: /UART_TX -> Net-(DD1-Pad15)
- DD1 pad 16: /UART_RX -> Net-(DD1-Pad16)
- DD1 pad 25: /ESP_IO0 -> Net-(DD1-Pad25)
- DD1 pad 26: /ESP_IO2 -> Net-(DD1-Pad26)
- DD1 pad 27: /ESP_CH_PD -> Net-(DD1-Pad27)
- DD1 pad 28: /ESP_REST -> Net-(DD1-Pad28)
Routing:
- net Net-(BQ1-Pad2): track 0.00 -> 4.76 mm
- net Net-(BQ1-Pad1): track 0.00 -> 4.76 mm
- net +3.3V: track 0.00 -> 1.95 mm
Other:
- board outline added: 61 x 41 mm
- board text added: "DISPLAY"
- board text added: "SENSOR"

Commit message: upd
Parts:
- added C2: 1 мкФ-NP0-16В ±5% 0805, Capacitor_SMD:C_0805_2012Metric, F.Cu at (64.8, 52.2)
- added DA2: BQ21040, Package_TO_SOT_SMD:SOT-23-6, F.Cu at (54.4, 64.4)
- added HL1: HL_LED, LED_SMD:LED_0603_1608Metric, F.Cu at (64.6, 55.0)
- added R12: 47 кОм ±5% 0603, Resistor_SMD:R_0603_1608Metric, F.Cu at (83.9, 76.4)
- added R2: 1,0 кОм ±1% 0603, Resistor_SMD:R_0603_1608Metric, F.Cu at (58.8, 63.4)
- added R4: 10 кОм ±5% 0603, Resistor_SMD:R_0603_1608Metric, F.Cu at (64.5, 57.6)
- added R6: 1,5 кОм ±5% 0603, Resistor_SMD:R_0603_1608Metric, F.Cu at (64.5, 60.1)
- added SA2: PTS645VM58-2 LFS, Button_Switch_THT:SW_Tactile_SPST_Angled_PTS645Vx58-2LFS, F.Cu at (55.0, 57.1)
- added XS4: 5.5x2.1, Connector_BarrelJack:BarrelJack_CUI_PJ-063AH_Horizontal, F.Cu at (45.4, 52.8)
- R9: renamed from R6; value 47 кОм ±5% 0603 -> 100 Ом ±5% 0603
- renumbered C2 to C3, C3 to C4, C4 to C5, C5 to C6, C6 to C7, C7 to C8, DA2 to DA3, R12 to R10, R13 to R11, R14 to R13, R15 to R14, R7 to R15, R9 to R16, R8 to R17, R10 to R18, R2 to R3, R3 to R5, R4 to R7, R5 to R8, VT2 to VT1, VT1 to VT2
Connections:
- C6 pad 1: Net-(C5-Pad1) -> Net-(C6-Pad1)
- DD1 pad 7: Net-(C5-Pad1) -> Net-(C6-Pad1)
- R9 pad 1: +3.3V -> EXP
- R9 pad 2: Net-(C5-Pad1) -> Net-(R9-Pad2)

Commit message: update
Parts:
- removed GB1: Battery_Cell, Battery:BatteryHolder_Keystone_2462_2xAA
- removed R9: 100 Ом ±5% 0603, Resistor_SMD:R_0603_1608Metric
- added REF**: MountingHole_2.2mm_M2_DIN965_Pad, MountingHole:MountingHole_2.2mm_M2_DIN965_Pad, F.Cu at (90.8, 68.0)
- added REF**: MountingHole_2.2mm_M2_DIN965_Pad, MountingHole:MountingHole_2.2mm_M2_DIN965_Pad, F.Cu at (106.2, 69.0)
- added REF**: MountingHole_3.2mm_M3_DIN965_Pad, MountingHole:MountingHole_3.2mm_M3_DIN965_Pad, F.Cu at (57.5, 49.8)
- added REF**: MountingHole_2.2mm_M2_DIN965_Pad, MountingHole:MountingHole_2.2mm_M2_DIN965_Pad, F.Cu at (56.2, 43.0)
- added REF**: MountingHole_2.2mm_M2_DIN965_Pad, MountingHole:MountingHole_2.2mm_M2_DIN965_Pad, F.Cu at (67.7, 44.5)
- added REF**: MountingHole_2.2mm_M2_DIN965_Pad, MountingHole:MountingHole_2.2mm_M2_DIN965_Pad, F.Cu at (67.7, 68.0)
- added REF**: MountingHole_2.2mm_M2_DIN965_Pad, MountingHole:MountingHole_2.2mm_M2_DIN965_Pad, F.Cu at (90.8, 44.5)
- added XP1: JST, Connector_JST:JST_SUR_BM02B-SURS-TF_1x02-1MP_P0.80mm_Vertical, B.Cu at (99.9, 43.6)
- SA1: footprint Button_Switch_THT:SW_Tactile_SPST_Angled_PTS645Vx58-2LFS -> Button_Switch_SMD:SW_Push_1P1T_NO_6x6mm_H9.5mm
- SA2: footprint Button_Switch_THT:SW_Tactile_SPST_Angled_PTS645Vx58-2LFS -> Button_Switch_SMD:SW_SPDT_PCM12; moved to B.Cu
- VT2: moved to B.Cu
- XS4: value 5.5x2.1 -> USB_A; footprint Connector_BarrelJack:BarrelJack_CUI_PJ-063AH_Horizontal -> Connector_USB:USB_Micro-B_Molex_47346-0001; moved to B.Cu
- moved XS4 60.3 mm to (105.7, 50.4), turned to -90 degrees
- moved SA2 51.3 mm to (106.2, 60.1), turned to -90 degrees
- moved SA1 49.5 mm to (60.0, 65.8)
- moved DD1 49.0 mm to (73.9, 53.6)
- moved BQ1 48.3 mm to (67.8, 52.4)
- moved DA3 42.8 mm to (64.0, 80.5)
- moved C4 40.0 mm to (71.4, 84.0)
- moved C3 40.0 mm to (68.4, 84.8)
- moved R1 38.0 mm to (70.0, 87.3)
- moved HL1 36.6 mm to (98.1, 69.7)
- moved XS1 32.7 mm to (100.5, 46.4), turned to -90 degrees
- moved L1 31.5 mm to (74.8, 80.6)
- moved XS2 30.3 mm to (56.1, 58.8)
- moved R5 29.5 mm to (75.6, 86.9)
- moved R7 29.5 mm to (74.8, 84.5)
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Connections:
- DA1 pad 1: Net-(DA1-Pad1) -> unconnected-(DA1-Pad1)
- DD1 pad 1: Net-(DD1-Pad1) -> unconnected-(DD1-Pad1)
- DD1 pad 10: Net-(DD1-Pad10) -> unconnected-(DD1-Pad10)
- DD1 pad 11: Net-(DD1-Pad11) -> unconnected-(DD1-Pad11)
- DD1 pad 14: Net-(DD1-Pad14) -> unconnected-(DD1-Pad14)
- DD1 pad 17: Net-(DD1-Pad17) -> unconnected-(DD1-Pad17)
- DD1 pad 18: Net-(DD1-Pad18) -> unconnected-(DD1-Pad18)
- DD1 pad 19: Net-(DD1-Pad19) -> unconnected-(DD1-Pad19)
- DD1 pad 20: Net-(DD1-Pad20) -> unconnected-(DD1-Pad20)
- DD1 pad 21: Net-(DD1-Pad21) -> unconnected-(DD1-Pad21)
- DD1 pad 22: Net-(DD1-Pad22) -> unconnected-(DD1-Pad22)
- DD1 pad 23: Net-(DD1-Pad23) -> unconnected-(DD1-Pad23)
- DD1 pad 3: Net-(DD1-Pad3) -> unconnected-(DD1-Pad3)
- DD1 pad 9: Net-(DD1-Pad9) -> unconnected-(DD1-Pad9)
- SA2 pad 1: Net-(C6-Pad1) -> Net-(SA2-Pad1)
- SA2 pad 2: Net-(R9-Pad2) -> Net-(SA2-Pad2)
- VT1 pad 3: Net-(GB1-Pad1) -> Net-(SA2-Pad2)
- XS4 pad 2: EXP -> unconnected-(XS4-Pad2)
Routing:
- net Net-(BQ1-Pad2): track 4.76 -> 0.00 mm
- net Net-(BQ1-Pad1): track 4.76 -> 0.00 mm
- net +3.3V: track 1.95 -> 0.00 mm
Other:
- board size 61 x 41 mm -> 54.2 x 30.3 mm
- net class Default removed

Commit message: pcb almost done
Parts:
- removed VT1: Si2307BDS, Package_TO_SOT_SMD:SOT-23
- C1, C2, C3, C4, C7, C8, DA1, DA2, DA3, HL1, L1, R1, R2, R3, R4, R6: moved to B.Cu
- XP1: footprint Connector_JST:JST_SUR_BM02B-SURS-TF_1x02-1MP_P0.80mm_Vertical -> Connector_PinHeader_2.54mm:PinHeader_1x02_P2.54mm_Vertical
- moved R6 66.5 mm to (106.2, 44.2), turned to 180 degrees
- moved R2 62.6 mm to (100.1, 45.3)
- moved DA2 62.4 mm to (98.2, 48.1)
- moved R18 61.2 mm to (85.6, 49.3), turned to 90 degrees
- moved R16 61.0 mm to (83.8, 48.2), turned to 90 degrees
- moved R17 59.0 mm to (65.6, 53.1)
- moved C2 58.6 mm to (101.5, 48.1), turned to 90 degrees
- moved R3 57.6 mm to (96.2, 54.0), turned to -90 degrees
- moved R4 57.1 mm to (99.2, 50.8)
- moved R15 48.9 mm to (67.5, 59.5), turned to 90 degrees
- moved C6 47.9 mm to (81.8, 48.9), turned to 90 degrees
- moved R14 44.9 mm to (88.8, 52.4)
- moved R1 44.3 mm to (95.0, 50.8), turned to 180 degrees
- moved R8 43.9 mm to (71.2, 64.4), turned to -90 degrees
- moved C5 43.7 mm to (75.0, 51.4), turned to 180 degrees
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Connections:
- C3 pad 1: Net-(C3-Pad1) -> Net-(SA2-Pad2)
- DA2 pad 2: Net-(C3-Pad1) -> Net-(DA2-Pad2)
- DA3 pad 5: Net-(C3-Pad1) -> Net-(SA2-Pad2)
- R1 pad 1: Net-(C3-Pad1) -> Net-(DA2-Pad2)
- R10 pad 1: /ESP_IO2 -> /ESP_REST
- R11 pad 1: /ESP_REST -> /ESP_CH_PD
- R14 pad 1: /ESP_CH_PD -> /ESP_IO2
- R5 pad 1: Net-(C3-Pad1) -> Net-(DA2-Pad2)
- R6 pad 2: Net-(C3-Pad1) -> Net-(DA2-Pad2)
- R7 pad 1: Net-(C3-Pad1) -> Net-(DA2-Pad2)
- REF** pad 1: (no net) -> EXP (x7)
- SA2 pad 1: Net-(SA2-Pad1) -> Net-(DA2-Pad2)
- XP1 pad 1: Net-(SA2-Pad1) -> Net-(DA2-Pad2)
Routing:
- net /SDA: track 0.00 -> 52.3 mm
- net /SCL: track 0.00 -> 44.5 mm
- net Net-(DD1-Pad24): track 0.00 -> 42.8 mm
- net +3.3V: track 0.00 -> 42.4 mm, vias 0 -> 5
- net Net-(DA2-Pad2): track 0.00 -> 38.9 mm, vias 0 -> 1
- net /UART_TX: track 0.00 -> 22.0 mm
- net /ESP_IO0: track 0.00 -> 21.1 mm
- net /ESP_IO2: track 0.00 -> 18.0 mm
- net Net-(DD1-Pad15): track 0.00 -> 13.6 mm
- net /UART_RX: track 0.00 -> 13.6 mm
- net /ESP_CH_PD: track 0.00 -> 13.1 mm
- net Net-(DD1-Pad16): track 0.00 -> 12.9 mm
- net Net-(DA2-Pad3): track 0.00 -> 11.5 mm
- net /BAT_ADC: track 0.00 -> 10.6 mm
- net Net-(C1-Pad2): track 0.00 -> 10.5 mm, vias 0 -> 2
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- added copper zone on B.Cu, net +3.3V
- added copper zone on B.Cu, net EXP
- added copper zone on F.Cu, net EXP
- added copper zone on B.Cu, net Net-(C1-Pad2)
- added copper zone on B.Cu, net Net-(C2-Pad1)
- added copper zone on B.Cu, net Net-(DA2-Pad2)
- added copper zone on B.Cu, net Net-(SA2-Pad2)
Other:
- board text removed: "DISPLAY"
