File: PCB/Curse_PCB/Curse_PCB.kicad_sch (KiCad schematic)
At the start: 41 parts

Commit message: pcb almost done
Parts:
- removed VT1: Si2307BDS, Package_TO_SOT_SMD:SOT-23, symbol Device_GOST:VT_PMOS_GSD
- XP1: footprint Connector_JST:JST_SUR_BM02B-SURS-TF_1x02-1MP_P0.80mm_Vertical -> Connector_PinHeader_2.54mm:PinHeader_1x02_P2.54mm_Vertical
Connections:
- net ESP_CH_PD: now also R11.1; no longer R14.1
- net ESP_IO2: now also R14.1; no longer R10.1
- net ESP_REST: now also R10.1; no longer R11.1
- net at DA2.2 (VOUT), R1.1, R5.1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: now also SA2.1, XP1.1; no longer C3.1, DA3.5 (VIN)
- net at SA2.2: now also C3.1, DA3.5 (VIN)
Other:
- moved on the sheet: SA2

Commit message: upd
Parts:
- removed XP1: JST, Connector_PinHeader_2.54mm:PinHeader_1x02_P2.54mm_Vertical, symbol Connector_Generic_GOST:CONN_2
- renumbered R11 to R10, R12 to R11, R13 to R12, R14 to R13, R15 to R14, R16 to R15, R17 to R16, R18 to R17, R10 to R9, SA2 to SA1, SA1 to SA2, VT2 to VT1
